File: filament-clock.kicad_pcb (KiCad board)
At the start: 2 copper layers, 66.6 x 94 mm, 51 parts, among them J1 UPDI, J2 Chain, SW1 h, SW2 m, U1 TLC59108xPW, U2 AP63203WU, U3 ATtiny412-SS, U4 PCF8523T, U5 apds-9006, Y1 32.768kHz

Commit message: Fix PCB
Parts:
- turned J1 to 180 degrees
- turned J2 to 90 degrees
